File: projects/pgiraude_project/pgiraude_project.kicad_sch (KiCad schematic)
At the start: 0 parts

Commit message: foot print
Parts:
- added C1, C2, C4, C5, C6, C7: ~, symbol my_library:capacitor_v2
- added C3: ~, symbol my_library:Crystal
- added D1, D2: ~, symbol my_library:Led
- added GND1, GND2, GND3, GND4, GND5, GND6, GND7, GND8: ~, symbol my_library:GND
- added J1: ~, symbol my_library:connector_1
- added J2: ~, symbol my_library:connector_2
- added J3: ~, symbol my_library:connector_3
- added R1, R2, R3: ~, symbol my_library:Resistor
- added SW_Push1: ~, symbol my_library:Sw_push
- added U1: ~, symbol my_library:atmega328p-A
Connections:
- new net: D1.2 (A), R1.2
- new net: C1.1, GND5.1
- new net: D1.1 (K), GND4.1
- new net: GND3.1, R2.2
- new net: C7.2, GND2.1
- new net: GND6.1, U1.3 (GND)
- new net: C3.1, C4.1, U1.7 (XTAL1/PB6)
- new net: C3.2, C4.2, C5.2, GND8.1
- new net: C6.2, GND1.1
- new net: C3.3, C5.1, U1.8 (XTAL2/PB7)
- new net: U1.18 (AVCC), U1.4 (VCC)
- new net: C2.2, U1.20 (AREF)
- new net: D2.1 (K), R2.1
- new net: C3.4, GND7.1
- new net: C1.2, SW_Push1.1
- new net A0: J2.8 (A0), U1.23 (PC0)
- new net A1: J2.7 (A1), U1.24 (PC1)
- new net A2: J2.6 (A2), U1.25 (PC2)
- new net A3: J2.5 (A3), U1.26 (PC3)
- new net A4: U1.27 (PC4)
- new net A5: U1.28 (PC5)
- new net A6: U1.19 (ADC6)
- new net A7: U1.22 (ADC7)
- new net D10: J2.12 (D10), U1.14 (PB2)
- new net D2: J1.8 (D2), U1.32 (PD2)
- new net D3: J1.7 (D3), U1.1 (PD3)
- new net D4: J1.6 (D4), U1.2 (PD4)
- new net D5: J1.5 (D5), U1.9 (PD5)
- new net D6: J1.4 (D6), U1.10 (PD6)
- new net D7: J1.3 (D7), U1.11 (PD7)
- new net D8: J1.2 (D8), U1.12 (PB0)
- new net D9: J1.1 (D9), U1.13 (PB1)
- new net DTR: J1.10 (RST), J2.3 (RST), J3.1 (DTR), R3.2, SW_Push1.2, U1.29 (RESET/PC6)
- new net GND: J1.9 (GND), J2.2 (GND), J3.5 (GND), J3.6 (GND)
- new net MISO: J2.10 (MISO), U1.16 (PB4)
- new net MOSI: J2.11 (MOSI), U1.15 (PB3)
- new net RAW: C6.1, C7.1, D2.2 (A), J2.1 (RAW)
- new net RXI: J1.11 (RXI), J3.3 (RXI), U1.30 (PD0)
- new net SCK: J2.9 (SCK), R1.1, U1.17 (PB5)
- new net TXO: J1.12 (TXO), J3.2 (TXO), U1.31 (PD1)
- new net VCC: J2.4 (VCC), J3.4 (VCC)

Commit message: pcb editor
Parts:
- added VCC1, VCC2, VCC3, VCC4: ~, symbol my_library:VCC
- ATmega1: renamed from U1; footprint (none) -> my_project:ATmega328-PAU
- C1: renamed from C5; value ~ -> 12pF; footprint (none) -> my_project:capacitor
- C2: renamed from C4; value ~ -> 12pF; footprint (none) -> my_project:capacitor
- C3: renamed from C2; value ~ -> 100nF; footprint (none) -> my_project:capacitor
- C4: renamed from C1; value ~ -> 100nF; footprint (none) -> my_project:capacitor
- C6: value ~ -> 1uF; footprint (none) -> my_project:capacitor
- C7: value ~ -> 100nF; footprint (none) -> my_project:capacitor
- D1: value ~ -> Green; footprint (none) -> my_project:led
- D2: value ~ -> Red; footprint (none) -> my_project:led
- GND1, GND2, GND3, GND4, GND5, GND6, GND7, GND8: now left out of the parts list
- J1: footprint (none) -> my_project:connector_1
- J2: footprint (none) -> my_project:connector_2
- J3: footprint (none) -> my_project:connector_3
- R1: value ~ -> 330; footprint (none) -> my_project:Resistor
- R2: footprint (none) -> my_project:Resistor
- R3: value ~ -> 10K; footprint (none) -> my_project:Resistor
- SW1: renamed from SW_Push1; value ~ -> SW_Push; footprint (none) -> my_project:switch
- Y1: renamed from C3; value ~ -> 16MHz; footprint (none) -> my_project:Crystal
Connections:
- net RAW: now also VCC1.
- net at R3.1: now also VCC4.
- net at ATmega1.18 (AVCC), ATmega1.4 (VCC): now also VCC2.
- net at C3.1: now also VCC3.
- no-connect marks 0 -> 4
Other:
- moved on the sheet: Y1
